File: KiCad/USB-TypeC-Switch.kicad_pcb (KiCad board)
At the start: 4 copper layers, 48.5 x 50 mm, 57 parts, among them J1 USB_C_IN_1, J2 USB_C_IN_2, J3 USB_C_OUT, J4 Conn_02x05_Odd_Even, SW1 SW_Push, U1 FUSB340TMX, U2 FUSB340TMX, U3 NL3S588, U4 AP63205WU, U5 UCS3205-E_Q8A, U6 UCS3205-E_Q8A, U7 NL3S588, U8 AZ1117C-3.3, U9 ATSAMD21E15B-M

Commit message: Silkscreen, Gerbers, Renders
Parts:
- added REF**: OSHW-Logo2_9.8x8mm_SilkScreen, Symbol:OSHW-Logo2_9.8x8mm_SilkScreen, B.Cu at (71.9, 99.8)
- added REF**: KiCad-Logo2_5mm_SilkScreen, Symbol:KiCad-Logo2_5mm_SilkScreen, B.Cu at (72.0, 124.5)
Routing:
- net /USB 2.0 and Misc Signal Switching/SBU1_1: track 73.6 -> 71.9 mm
- net /USB 2.0 and Misc Signal Switching/D_2_N: track 48.5 -> 47.4 mm
- net /USB 2.0 and Misc Signal Switching/D_1_P: track 30.6 -> 31.7 mm
- net /USB 2.0 and Misc Signal Switching/SBU1: track 16.8 -> 15.9 mm
- net +3V3: track 213.9 -> 213.0 mm
- net /USB 2.0 and Misc Signal Switching/SBU1_2: track 30.3 -> 30.5 mm, vias 4 -> 6
- net /USB 2.0 and Misc Signal Switching/SBU2_1: track 73.3 -> 73.2 mm, vias 3 -> 1
Other:
- board text added: "Designed by: Attila Tőkés (tokes_atti@yahoo.com)"
- board text added: "GitHub: bluetiger9/USB-Type-C-Switch"
- board text added: "Hackster.io: bluetiger9/usb-3-x-type-c-switch-0ceea6"
- board text added: "JLCJLCJLCJLC"
- board text added: "License: CC BY 4.0 (Attribution 4.0 Intl.)"
- board text added: "Revision: 1.0"
- board text added: "USB 3.x Type-C Switch"

Commit message: Migrate to KiCad 6.x
Other:
- net class Default removed
- net class GNDS removed
- net class USB2_90ohm removed
- net class USB3_90ohm removed
- net class VBUS removed
- net class low_speed_diff removed
