File: KiCad/USB-TypeC-Switch.kicad_pcb (KiCad board)
At the start: 4 copper layers, 48.5 x 50 mm, 59 parts, among them J1 USB_C_IN_1, J2 USB_C_IN_2, J3 USB_C_OUT, J4 Conn_02x05_Odd_Even, SW1 SW_Push, U1 FUSB340TMX, U2 FUSB340TMX, U3 NL3S588, U4 AP63205WU, U5 UCS3205-E_Q8A, U6 UCS3205-E_Q8A, U7 NL3S588, U8 AZ1117C-3.3, U9 ATSAMD21E15B-M

Commit message: Fix USB 2.0 signal polarity (+others)
Connections:
- net /USB 2.0 and Misc Signal Switching/D_2_N renamed /Control/D_N_uC
- net /USB 2.0 and Misc Signal Switching/D_2_P renamed /Control/D_P_uC
- net /USB 2.0 and Misc Signal Switching/SEL renamed /Control/SEL_USB2_SBU
- net /USB 3 Signal Switching/OE_N renamed /Control/OE_N_USB3
- net /USB 3 Signal Switching/SEL renamed /Control/SEL_USB3
- J3 pad A6: /USB 2.0 and Misc Signal Switching/D_N -> /USB 2.0 and Misc Signal Switching/D_P
- J3 pad A7: /USB 2.0 and Misc Signal Switching/D_P -> /USB 2.0 and Misc Signal Switching/D_N
- J3 pad B6: /USB 2.0 and Misc Signal Switching/D_N -> /USB 2.0 and Misc Signal Switching/D_P
- J3 pad B7: /USB 2.0 and Misc Signal Switching/D_P -> /USB 2.0 and Misc Signal Switching/D_N
- J4 pad 6: (no net) -> unconnected-(J4-Pad6)
- J4 pad 8: (no net) -> unconnected-(J4-Pad8)
- S1 pad 1: (no net) -> unconnected-(S1-Pad1)
- S1 pad 13: (no net) -> unconnected-(S1-Pad13)
- S1 pad 5: (no net) -> unconnected-(S1-Pad5)
- S1 pad 9: (no net) -> unconnected-(S1-Pad9)
- U5 pad 10: (no net) -> unconnected-(U5-Pad10)
- U5 pad 11: (no net) -> unconnected-(U5-Pad11)
- U5 pad 6: (no net) -> unconnected-(U5-Pad6)
- U5 pad 7: (no net) -> unconnected-(U5-Pad7)
- U5 pad 8: (no net) -> unconnected-(U5-Pad8)
- U5 pad 9: (no net) -> unconnected-(U5-Pad9)
- U6 pad 10: (no net) -> unconnected-(U6-Pad10)
- U6 pad 11: (no net) -> unconnected-(U6-Pad11)
- U6 pad 6: (no net) -> unconnected-(U6-Pad6)
- U6 pad 7: (no net) -> unconnected-(U6-Pad7)
- U6 pad 8: (no net) -> unconnected-(U6-Pad8)
- U6 pad 9: (no net) -> unconnected-(U6-Pad9)
- U9 pad 13: (no net) -> unconnected-(U9-Pad13)
- U9 pad 14: (no net) -> unconnected-(U9-Pad14)
- U9 pad 2: (no net) -> unconnected-(U9-Pad2)
- U9 pad 22: (no net) -> unconnected-(U9-Pad22)
- U9 pad 27: (no net) -> unconnected-(U9-Pad27)
- U9 pad 33: (no net) -> unconnected-(U9-Pad33)
- U9 pad 8: (no net) -> unconnected-(U9-Pad8)
Routing:
- net GNDS: track 457.0 -> 41.3 mm
- net GND: track 77.2 -> 76.7 mm
- net /USB 2.0 and Misc Signal Switching/D_P: track 15.2 -> 15.4 mm, vias 2 -> 3
- net /USB 2.0 and Misc Signal Switching/D_N: track 15.3 -> 15.4 mm, vias 3 -> 2
- net /Control/SEL_USB2_SBU: vias 3 -> 2
- added copper zone on B.Cu, net GNDS
- added copper zone on F.Cu, net GNDS

Commit message: Use 0603 resistors and capacitors
Parts:
- C1, C4, C5, C6, C7, C9: footprint Capacitor_SMD:C_0805_2012Metric -> Capacitor_SMD:C_0603_1608Metric
- R1, R10, R13, R14, R15, R16, R17, R18, R19, R2, R23, R3, R4, R5, R6, R9: footprint Resistor_SMD:R_0805_2012Metric -> Resistor_SMD:R_0603_1608Metric

Commit message: 6 layers
Routing:
- added copper zone on In4.Cu, net GND
- removed copper zone on In2.Cu, net GND
Other:
- copper layers 4 -> 6
Changed lines of the file:
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@@
 (kicad_pcb (version 20211014) (generator pcbnew)
   (general
-    (thickness 1.6)
+    (thickness 1.5584)
   )
   (paper "A4")
@@
     (1 "In1.Cu" power)
     (2 "In2.Cu" power)
+    (3 "In3.Cu" signal)
+    (4 "In4.Cu" signal)
     (31 "B.Cu" signal)
     (32 "B.Adhes" user "B.Adhesive")
@@
       (layer "F.Mask" (type "Top Solder Mask") (thickness 0.01))
       (layer "F.Cu" (type "copper") (thickness 0.035))
-      (layer "dielectric 1" (type "core") (thickness 0.48) (material "FR4") (epsilon_r 4.5) (loss_tangent 0.02))
-      (layer "In1.Cu" (type "copper") (thickness 0.035))
-      (layer "dielectric 2" (type "prepreg") (thickness 0.48) (material "FR4") (epsilon_r 4.5) (loss_tangent 0.02))
-      (layer "In2.Cu" (type "copper") (thickness 0.035))
-      (layer "dielectric 3" (type "core") (thickness 0.48) (material "FR4") (epsilon_r 4.5) (loss_tangent 0.02))
+      (layer "dielectric 1" (type "prepreg") (thickness 0.0994) (material "JLC-3313") (epsilon_r 4.05) (loss_tangent 0.02))
+      (layer "In1.Cu" (type "copper") (thickness 0.0152))
+      (layer "dielectric 2" (type "core") (thickness 0.55) (material "JLC-Core") (epsilon_r 4.6) (loss_tangent 0.02))
+      (layer "In2.Cu" (type "copper") (thickness 0.0152))
+      (layer "dielectric 3" (type "prepreg") (thickness 0.1088) (material "JLC-2116") (epsilon_r 4.25) (loss_tangent 0.02))
+      (layer "In3.Cu" (type "copper") (thickness 0.0152))
+      (layer "dielectric 4" (type "core") (thickness 0.55) (material "JLC-Core") (epsilon_r 4.6) (loss_tangent 0.02))
+      (layer "In4.Cu" (type "copper") (thickness 0.0152))
+      (layer "dielectric 5" (type "prepreg") (thickness 0.0994) (material "JLC-3313") (epsilon_r 4.05) (loss_tangent 0.02))
       (layer "B.Cu" (type "copper") (thickness 0.035))
       (layer "B.Mask" (type "Bottom Solder Mask") (thickness 0.01))
@@
       (layer "B.SilkS" (type "Bottom Silk Screen"))
       (copper_finish "None")
-      (dielectric_constraints no)
+      (dielectric_constraints yes)
     )
     (pad_to_mask_clearance 0)
@@
     )
   )
-  (zone (net 3) (net_name "GND") (layers "In1.Cu" "In2.Cu") (hatch edge 0.508)
-    (connect_pads (clearance 0.2))
-    (min_thickness 0.254) (filled_areas_thickness no)
-    (fill yes (thermal_gap 0.508) (thermal_bridge_width 0.508))
-    (polygon
-      (pts
-        (xy 79.29 136.04)
-        (xy 30.7 136.04)
-        (xy 30.71 85.96)
-        (xy 79.27 85.97)
-      )
-    )
-  )
-  (zone (net 3) (net_name "GND") (layer "In2.Cu") (hatch edge 0.508)
+  (zone (net 3) (net_name "GND") (layers "In1.Cu" "In4.Cu") (hatch edge 0.508)
     (connect_pads (clearance 0.2))
     (min_thickness 0.254) (filled_areas_thickness no)

Commit message: 6 layers partial routing
Routing:
- net /USB 2.0 and Misc Signal Switching/SBU1_1: track 71.9 -> 35.7 mm
- net /USB 2.0 and Misc Signal Switching/SBU2_1: track 73.0 -> 40.7 mm
- net /USB 2.0 and Misc Signal Switching/CC1_1: track 83.6 -> 53.4 mm, vias 6 -> 2
- net /USB 2.0 and Misc Signal Switching/CC2_1: track 96.2 -> 66.5 mm, vias 3 -> 1
- net /Power Switching and Supplies/VBUS: track 29.8 -> 6.18 mm
- net /Power Switching and Supplies/VBUS_1: track 23.5 -> 2.66 mm
- net /Power Switching and Supplies/VBUS_2: track 26.3 -> 7.37 mm, vias 12 -> 4
- net +3V3: track 213.0 -> 194.4 mm, vias 15 -> 17
- net /USB 2.0 and Misc Signal Switching/CC2_2: track 30.2 -> 45.2 mm, vias 3 -> 1
- net /USB 2.0 and Misc Signal Switching/SBU1: track 15.9 -> 12.0 mm
- net /USB 2.0 and Misc Signal Switching/SBU1_2: track 30.5 -> 27.1 mm, vias 6 -> 2
- net /USB 2.0 and Misc Signal Switching/SBU2_2: track 35.6 -> 36.9 mm
- net GND: vias 132 -> 131
- added copper zone on In2.Cu, net +3V3
- added copper zone on In2.Cu, net /Power Switching and Supplies/VBUS
- added copper zone on In3.Cu, net /Power Switching and Supplies/VBUS
- added copper zone on F.Cu, net /Power Switching and Supplies/VBUS_1
- added copper zone on In2.Cu, net /Power Switching and Supplies/VBUS_1
- added copper zone on In3.Cu, net /Power Switching and Supplies/VBUS_1
- added copper zone on In2.Cu, net /Power Switching and Supplies/VBUS_2
- added copper zone on In3.Cu, net /Power Switching and Supplies/VBUS_2
- added copper zone on In2.Cu, net /Power Switching and Supplies/VBUS_OUT_FUSED
- added copper zone on In3.Cu, net /Power Switching and Supplies/VBUS_OUT_FUSED

Commit message: CC detect trigger + inner layer routing
Parts:
- added D7: 3.3V, Diode_SMD:D_SOD-523, F.Cu at (57.9, 89.8)
- added D8: 3.3V, Diode_SMD:D_SOD-523, F.Cu at (62.5, 89.7)
- added D9: 3.3V, Diode_SMD:D_SOD-523, F.Cu at (56.4, 89.8)
- added Q1: 2N7002, Package_DFN_QFN:Diodes_DFN1006-3, F.Cu at (67.8, 124.1)
- added Q2: 2N7002, Package_DFN_QFN:Diodes_DFN1006-3, F.Cu at (62.4, 124.1)
- added Q3: 2N7002, Package_DFN_QFN:Diodes_DFN1006-3, F.Cu at (65.1, 124.1)
- added Q4: 2N7002, Package_DFN_QFN:Diodes_DFN1006-3, F.Cu at (69.0, 124.1)
- added Q5: 2N7002, Package_DFN_QFN:Diodes_DFN1006-3, F.Cu at (63.6, 124.1)
- added Q6: 2N7002, Package_DFN_QFN:Diodes_DFN1006-3, F.Cu at (66.3, 124.1)
- added R11: 5.1k, Resistor_SMD:R_0402_1005Metric, F.Cu at (66.2, 125.9)
- added R12: 5.1k, Resistor_SMD:R_0402_1005Metric, F.Cu at (62.2, 125.9)
- added R20: 220k, Resistor_SMD:R_0402_1005Metric, F.Cu at (68.2, 125.9)
- added R21: 220k, Resistor_SMD:R_0402_1005Metric, F.Cu at (64.2, 125.9)
- added R22: 5.1k, Resistor_SMD:R_0402_1005Metric, F.Cu at (64.7, 122.7)
- added R24: 5.1k, Resistor_SMD:R_0402_1005Metric, F.Cu at (69.2, 125.9)
- added R25: 5.1k, Resistor_SMD:R_0402_1005Metric, F.Cu at (65.2, 125.9)
- added R26: 5.1k, Resistor_SMD:R_0402_1005Metric, F.Cu at (66.7, 122.7)
- added R27: 220k, Resistor_SMD:R_0402_1005Metric, F.Cu at (62.7, 122.7)
- added R28: 220k, Resistor_SMD:R_0402_1005Metric, F.Cu at (68.7, 122.7)
- added R7: 220k, Resistor_SMD:R_0402_1005Metric, F.Cu at (67.2, 125.9)
- added R8: 220k, Resistor_SMD:R_0402_1005Metric, F.Cu at (63.2, 125.9)
- moved S1 5.12 mm to (57.7, 124.3)
- moved F3 3.72 mm to (71.9, 119.8)
- moved D3 2.87 mm to (72.2, 125.0), turned to 90 degrees
- moved R18 2.51 mm to (76.3, 127.8), turned to 90 degrees
- moved D6 2.39 mm to (75.3, 117.3)
- moved R2 2.22 mm to (76.4, 120.1)
- moved R17 1.47 mm to (76.3, 124.5), turned to 90 degrees
- moved C7 0.50 mm to (59.4, 90.0)
Connections:
- U9 pad 13: unconnected-(U9-Pad13) -> /Control/PU_CC_2
- U9 pad 14: unconnected-(U9-Pad14) -> /Control/PU_CC
- U9 pad 8: unconnected-(U9-Pad8) -> /Control/PU_CC_1
Routing:
- net /Control/PU_CC: track 0.00 -> 63.5 mm, vias 0 -> 5
- net /Control/PU_CC_1: track 0.00 -> 57.8 mm, vias 0 -> 2
- net /Power Switching and Supplies/VBUS_OUT_FUSED: track 78.9 -> 21.6 mm
- net /Control/PU_CC_2: track 0.00 -> 56.1 mm, vias 0 -> 3
- net +3V3: track 194.4 -> 214.3 mm, vias 17 -> 12
- net /USB 2.0 and Misc Signal Switching/CC2_1: track 66.5 -> 51.5 mm, vias 1 -> 3
- net /USB 2.0 and Misc Signal Switching/CC1_2: track 27.3 -> 35.3 mm, vias 2 -> 4
- net /USB 2.0 and Misc Signal Switching/CC1_1: track 53.4 -> 45.5 mm
- net GND: track 76.6 -> 83.3 mm, vias 131 -> 136
- net /USB 2.0 and Misc Signal Switching/CC1: track 25.4 -> 32.1 mm, vias 2 -> 3
- net /Control/OE_CC_1: track 51.1 -> 57.4 mm
- net +5V: track 19.5 -> 14.4 mm
- net /Control/OE_CC_2: track 55.7 -> 58.8 mm
- net Net-(Q5-Pad3): track 0.00 -> 1.96 mm
- net Net-(Q1-Pad3): track 0.00 -> 1.96 mm
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- removed copper zone on In2.Cu, net +3V3
- removed copper zone on B.Cu, net /Power Switching and Supplies/VBUS_OUT_FUSED

Commit message: 6 layer re-routing
Parts:
- added R29: 220k, Resistor_SMD:R_0603_1608Metric, F.Cu at (48.4, 92.5)
- added R30: 220k, Resistor_SMD:R_0603_1608Metric, F.Cu at (51.6, 92.5)
- added R31: 220k, Resistor_SMD:R_0603_1608Metric, F.Cu at (75.4, 122.2)
- moved D8 6.55 mm to (56.0, 90.4)
- moved R2 3.16 mm to (75.9, 117.0), turned to 0 degrees
- moved R18 2.73 mm to (75.4, 125.2), turned to 0 degrees
- moved R17 2.54 mm to (75.4, 126.8), turned to 180 degrees
- moved D9 2.12 mm to (54.4, 90.4)
- moved R6 2.12 mm to (57.5, 97.0), turned to -45 degrees
- moved R5 1.96 mm to (48.5, 89.9), turned to 180 degrees
- moved D3 1.94 mm to (71.2, 123.4)
- moved D6 1.60 mm to (75.7, 118.8)
- moved R4 1.38 mm to (51.6, 89.9), turned to 180 degrees
- moved C4 1.16 mm to (68.2, 99.1)
- moved F3 1.03 mm to (71.1, 119.2)
- moved Q1 0.97 mm to (66.8, 124.2)
- moved Q2 0.97 mm to (61.4, 124.2)
- moved Q3 0.97 mm to (64.1, 124.2)
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Connections:
- net /Control/D_N_uC renamed /Control/D_uC_N
- net /Control/D_P_uC renamed /Control/D_uC_P
Routing:
- net +3V3: track 214.3 -> 146.4 mm, vias 12 -> 10
- net /Control/SEL_USB2_SBU: track 60.3 -> 25.2 mm
- net /Control/OE_N_SBU: track 49.4 -> 32.9 mm
- net /Control/OE_CC_1: track 57.4 -> 44.9 mm
- net Net-(J4-Pad10): track 23.9 -> 12.7 mm
- net /Control/OE_CC_2: track 58.8 -> 47.9 mm
- net /Power Switching and Supplies/VBUS_IN2_FUSED: track 59.5 -> 69.0 mm
- net GND: track 83.3 -> 75.5 mm, vias 136 -> 145
- net /Power Switching and Supplies/VBUS_IN1_FUSED: track 38.7 -> 46.1 mm
- net Net-(SW1-Pad2): track 20.4 -> 14.1 mm
- net /Control/PU_CC_1: track 57.8 -> 63.4 mm, vias 2 -> 3
- net /Control/LED_OUT: track 35.4 -> 30.6 mm
- net /USB 2.0 and Misc Signal Switching/CC1_1: track 45.5 -> 40.7 mm
- net /Control/SWDCLK: track 17.5 -> 13.3 mm, vias 3 -> 2
- net /Control/OE_PWR_2: track 54.8 -> 50.7 mm, vias 2 -> 3
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- added copper zone on In2.Cu, net GND
- added copper zone on In3.Cu, net GND

Commit message: resistor value + stitching vias
Parts:
- D7, D8, D9: value 3.3V -> 3.6V
- Q1, Q2, Q3, Q4, Q5, Q6: value 2N7002 -> AP1606
- R1, R2, R3: value 220 -> 470
- R13, R15, R17: value 9k -> 47k
- R14, R16, R18: value 1k -> 5.6k
- R4, R5: value 9k -> 10k
- renumbered REF** to REF_KICAD_LOGO, REF** to REF_OSH_LOGO_1, REF** to REF_OSH_LOGO_2
Routing:
- net GND: vias 145 -> 165
- net /Power Switching and Supplies/VBUS_OUT_FUSED: vias 15 -> 18
Other:
- board text added: "Revision: 1.1"
- board text removed: "Revision: 1.0"

Commit message: 6 layer 1.6mm stackup + gerbers + bom + position files
Routing:
- net /USB 2.0 and Misc Signal Switching/SBU1_2: track 27.1 -> 34.3 mm
- net /USB 2.0 and Misc Signal Switching/SBU1_1: track 34.5 -> 41.6 mm
- net /USB 2.0 and Misc Signal Switching/SBU1: track 13.0 -> 17.2 mm
- net /USB 2.0 and Misc Signal Switching/SBU2: track 19.7 -> 18.3 mm
- net /Control/PU_CC: track 64.6 -> 63.9 mm
- net GND: vias 165 -> 168
