File: KiCad/USB-TypeC-Switch.kicad_sch (KiCad schematic)
At the start: 9 parts, among them J1 USB_C_IN_1, J2 USB_C_IN_2, J3 USB_C_OUT

Commit message: Fix USB 2.0 signal polarity (+others)
Connections:
- net USB 2.0 and Misc Signal Switching/D_N: now also J3.A7 (D-), J3.B7 (D-); no longer J3.A6 (D+), J3.B6 (D+)
- net USB 2.0 and Misc Signal Switching/D_P: now also J3.A6 (D+), J3.B6 (D+); no longer J3.A7 (D-), J3.B7 (D-)
Changed lines of the file:
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@@
-    (stroke (width 0) (type default) (color 0 0 0 0))
-  )
-  (wire (pts (xy 194.31 64.77) (xy 245.11 64.77))
     (stroke (width 0) (type default) (color 0 0 0 0))
   )
@@
     (stroke (width 0) (type default) (color 0 0 0 0))
   )
-  (wire (pts (xy 138.43 46.99) (xy 196.85 46.99))
-    (stroke (width 0) (type default) (color 0 0 0 0))
-  )
   (wire (pts (xy 57.15 39.37) (xy 57.15 116.84))
     (stroke (width 0) (type default) (color 0 0 0 0))
@@
     (stroke (width 0) (type default) (color 0 0 0 0))
   )
+  (wire (pts (xy 138.43 46.99) (xy 196.215 46.99))
+    (stroke (width 0) (type default) (color 0 0 0 0))
+  )
   (wire (pts (xy 147.32 22.86) (xy 138.43 22.86))
     (stroke (width 0) (type default) (color 0 0 0 0))
@@
     (stroke (width 0) (type default) (color 0 0 0 0))
   )
+  (wire (pts (xy 196.215 64.77) (xy 245.11 64.77))
+    (stroke (width 0) (type default) (color 0 0 0 0))
+  )
   (wire (pts (xy 68.58 134.62) (xy 40.64 134.62))
     (stroke (width 0) (type default) (color 0 0 0 0))
@@
     (stroke (width 0) (type default) (color 0 0 0 0))
   )
-  (wire (pts (xy 194.31 49.53) (xy 194.31 64.77))
+  (wire (pts (xy 194.31 49.53) (xy 194.31 62.23))
     (stroke (width 0) (type default) (color 0 0 0 0))
   )
@@
     (stroke (width 0) (type default) (color 0 0 0 0))
   )
-  (wire (pts (xy 196.85 46.99) (xy 196.85 62.23))
-    (stroke (width 0) (type default) (color 0 0 0 0))
-  )
   (wire (pts (xy 45.72 31.75) (xy 45.72 34.29))
     (stroke (width 0) (type default) (color 0 0 0 0))
@@
     (stroke (width 0) (type default) (color 0 0 0 0))
   )
+  (wire (pts (xy 196.215 46.99) (xy 196.215 64.77))
+    (stroke (width 0) (type default) (color 0 0 0 0))
+  )
   (wire (pts (xy 48.26 82.55) (xy 91.44 82.55))
     (stroke (width 0) (type default) (color 0 0 0 0))
@@
     (stroke (width 0) (type default) (color 0 0 0 0))
   )
-  (wire (pts (xy 196.85 62.23) (xy 245.11 62.23))
-    (stroke (width 0) (type default) (color 0 0 0 0))
-  )
+  (wire (pts (xy 194.31 62.23) (xy 245.11 62.23))
+    (stroke (width 0) (type default) (color 0 0 0 0))
+  )

Commit message: Use 0603 resistors and capacitors
Parts:
- C9: footprint Capacitor_SMD:C_0805_2012Metric -> Capacitor_SMD:C_0603_1608Metric
- R23: footprint Resistor_SMD:R_0805_2012Metric -> Resistor_SMD:R_0603_1608Metric
Changed lines of the file:
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@@
     (property "Reference" "C9" (id 0) (at 267.97 120.65 90))
     (property "Value" "100n" (id 1) (at 267.97 128.27 90))
-    (property "Footprint" "Capacitor_SMD:C_0805_2012Metric" (id 2) (at 267.97 124.46 0)
+    (property "Footprint" "Capacitor_SMD:C_0603_1608Metric" (id 2) (at 267.97 124.46 0)
       (effects (font (size 1.27 1.27)) hide)
     )
@@
     (property "Reference" "R23" (id 0) (at 267.97 113.03 90))
     (property "Value" "100k" (id 1) (at 267.97 118.11 90))
-    (property "Footprint" "Resistor_SMD:R_0805_2012Metric" (id 2) (at 267.97 115.57 0)
+    (property "Footprint" "Resistor_SMD:R_0603_1608Metric" (id 2) (at 267.97 115.57 0)
       (effects (font (size 1.27 1.27)) hide)
     )
@@
     )
     (property "Sheet file" "h_usb3_switching.kicad_sch" (id 1) (at 104.14 145.3646 0)
-      (effects (font (size 1.27 1.27)) (justify left top))
+      (effects (font (size 1.27 1.27)) (justify left top) hide)
     )
     (pin "RX1_1_N" input (at 104.14 101.6 180)
@@
     )
     (property "Sheet file" "h_usb2_misc.kicad_sch" (id 1) (at 104.14 84.4046 0)
-      (effects (font (size 1.27 1.27)) (justify left top))
+      (effects (font (size 1.27 1.27)) (justify left top) hide)
     )
     (pin "D_1_P" input (at 104.14 46.99 180)
@@
     )
     (property "Sheet file" "h_power.kicad_sch" (id 1) (at 104.14 37.4146 0)
-      (effects (font (size 1.27 1.27)) (justify left top))
+      (effects (font (size 1.27 1.27)) (justify left top) hide)
     )
     (pin "VBUS_1" input (at 104.14 19.05 180)
@@
     )
     (property "Sheet file" "h_control.kicad_sch" (id 1) (at 104.14 191.0846 0)
-      (effects (font (size 1.27 1.27)) (justify left top))
+      (effects (font (size 1.27 1.27)) (justify left top) hide)
     )
     (pin "OE_PWR_1" output (at 138.43 161.29 0)
@@
     )
     (path "/00000000-0000-0000-0000-00006086b3f3/00000000-0000-0000-0000-000060f18943"
-      (reference "C1") (unit 1) (value "100n") (footprint "Capacitor_SMD:C_0805_2012Metric")
+      (reference "C1") (unit 1) (value "100n") (footprint "Capacitor_SMD:C_0603_1608Metric")
     )
     (path "/00000000-0000-0000-0000-00006086b3f3/00000000-0000-0000-0000-000060f53ead"
@@
     )
     (path "/00000000-0000-0000-0000-0000610e53f5/00000000-0000-0000-0000-000061543d7b"
-      (reference "C4") (unit 1) (value "1u") (footprint "Capacitor_SMD:C_0805_2012Metric")
+      (reference "C4") (unit 1) (value "1u") (footprint "Capacitor_SMD:C_0603_1608Metric")
     )
     (path "/00000000-0000-0000-0000-0000610e53f5/00000000-0000-0000-0000-000061544cdd"
-      (reference "C5") (unit 1) (value "100n") (footprint "Capacitor_SMD:C_0805_2012Metric")
+      (reference "C5") (unit 1) (value "100n") (footprint "Capacitor_SMD:C_0603_1608Metric")
     )
     (path "/00000000-0000-0000-0000-0000610e53f5/00000000-0000-0000-0000-00006191a7d7"
-      (reference "C6") (unit 1) (value "100n") (footprint "Capacitor_SMD:C_0805_2012Metric")
+      (reference "C6") (unit 1) (value "100n") (footprint "Capacitor_SMD:C_0603_1608Metric")
     )
     (path "/00000000-0000-0000-0000-0000610e53f5/00000000-0000-0000-0000-00006191a7d1"
-      (reference "C7") (unit 1) (value "1u") (footprint "Capacitor_SMD:C_0805_2012Metric")
+      (reference "C7") (unit 1) (value "1u") (footprint "Capacitor_SMD:C_0603_1608Metric")
     )
     (path "/00000000-0000-0000-0000-00006086b3f3/00000000-0000-0000-0000-0000601a67ea"
@@
     )
     (path "/00000000-0000-0000-0000-0000601df1ae"
-      (reference "C9") (unit 1) (value "100n") (footprint "Capacitor_SMD:C_0805_2012Metric")
+      (reference "C9") (unit 1) (value "100n") (footprint "Capacitor_SMD:C_0603_1608Metric")
     )
     (path "/00000000-0000-0000-0000-00006086b3f3/00000000-0000-0000-0000-0000602bd916"
@@
     )
     (path "/00000000-0000-0000-0000-0000610e53f5/00000000-0000-0000-0000-000060142a37"
-      (reference "R1") (unit 1) (value "220") (footprint "Resistor_SMD:R_0805_2012Metric")
+      (reference "R1") (unit 1) (value "220") (footprint "Resistor_SMD:R_0603_1608Metric")
     )
     (path "/00000000-0000-0000-0000-0000610e53f5/00000000-0000-0000-0000-000060140919"
-      (reference "R2") (unit 1) (value "220") (footprint "Resistor_SMD:R_0805_2012Metric")
+      (reference "R2") (unit 1) (value "220") (footprint "Resistor_SMD:R_0603_1608Metric")
     )
     (path "/00000000-0000-0000-0000-0000610e53f5/00000000-0000-0000-0000-0000616a374f"
-      (reference "R3") (unit 1) (value "220") (footprint "Resistor_SMD:R_0805_2012Metric")
+      (reference "R3") (unit 1) (value "220") (footprint "Resistor_SMD:R_0603_1608Metric")
     )
     (path "/00000000-0000-0000-0000-00006086b3f3/00000000-0000-0000-0000-0000600bbec3"
-      (reference "R4") (unit 1) (value "9k") (footprint "Resistor_SMD:R_0805_2012Metric")
+      (reference "R4") (unit 1) (value "9k") (footprint "Resistor_SMD:R_0603_1608Metric")
     )
     (path "/00000000-0000-0000-0000-00006086b3f3/00000000-0000-0000-0000-0000600c3d30"
-      (reference "R5") (unit 1) (value "9k") (footprint "Resistor_SMD:R_0805_2012Metric")
+      (reference "R5") (unit 1) (value "9k") (footprint "Resistor_SMD:R_0603_1608Metric")
     )
     (path "/00000000-0000-0000-0000-00006060e5e3/00000000-0000-0000-0000-00006012d6cb"
-      (reference "R6") (unit 1) (value "10k") (footprint "Resistor_SMD:R_0805_2012Metric")
+      (reference "R6") (unit 1) (value "10k") (footprint "Resistor_SMD:R_0603_1608Metric")
     )
     (path "/00000000-0000-0000-0000-00006086b3f3/00000000-0000-0000-0000-000060e997de"
-      (reference "R9") (unit 1) (value "470") (footprint "Resistor_SMD:R_0805_2012Metric")
+      (reference "R9") (unit 1) (value "470") (footprint "Resistor_SMD:R_0603_1608Metric")
     )
     (path "/00000000-0000-0000-0000-00006086b3f3/00000000-0000-0000-0000-000060ea33cb"
-      (reference "R10") (unit 1) (value "470") (footprint "Resistor_SMD:R_0805_2012Metric")
+      (reference "R10") (unit 1) (value "470") (footprint "Resistor_SMD:R_0603_1608Metric")
     )
     (path "/00000000-0000-0000-0000-00006086b3f3/00000000-0000-0000-0000-00006156ae26"
-      (reference "R13") (unit 1) (value "9k") (footprint "Resistor_SMD:R_0805_2012Metric")
+      (reference "R13") (unit 1) (value "9k") (footprint "Resistor_SMD:R_0603_1608Metric")
     )
     (path "/00000000-0000-0000-0000-00006086b3f3/00000000-0000-0000-0000-00006156ae2c"
-      (reference "R14") (unit 1) (value "1k") (footprint "Resistor_SMD:R_0805_2012Metric")
+      (reference "R14") (unit 1) (value "1k") (footprint "Resistor_SMD:R_0603_1608Metric")
     )
     (path "/00000000-0000-0000-0000-00006086b3f3/00000000-0000-0000-0000-0000615833ba"
-      (reference "R15") (unit 1) (value "9k") (footprint "Resistor_SMD:R_0805_2012Metric")
+      (reference "R15") (unit 1) (value "9k") (footprint "Resistor_SMD:R_0603_1608Metric")
     )
     (path "/00000000-0000-0000-0000-00006086b3f3/00000000-0000-0000-0000-0000615833c0"
-      (reference "R16") (unit 1) (value "1k") (footprint "Resistor_SMD:R_0805_2012Metric")
+      (reference "R16") (unit 1) (value "1k") (footprint "Resistor_SMD:R_0603_1608Metric")
     )
     (path "/00000000-0000-0000-0000-00006086b3f3/00000000-0000-0000-0000-00006158fd1f"
-      (reference "R17") (unit 1) (value "9k") (footprint "Resistor_SMD:R_0805_2012Metric")
+      (reference "R17") (unit 1) (value "9k") (footprint "Resistor_SMD:R_0603_1608Metric")
     )
     (path "/00000000-0000-0000-0000-00006086b3f3/00000000-0000-0000-0000-00006158fd25"
-      (reference "R18") (unit 1) (value "1k") (footprint "Resistor_SMD:R_0805_2012Metric")
+      (reference "R18") (unit 1) (value "1k") (footprint "Resistor_SMD:R_0603_1608Metric")
     )
     (path "/00000000-0000-0000-0000-0000610e53f5/00000000-0000-0000-0000-000061664e03"
-      (reference "R19") (unit 1) (value "1k") (footprint "Resistor_SMD:R_0805_2012Metric")
+      (reference "R19") (unit 1) (value "1k") (footprint "Resistor_SMD:R_0603_1608Metric")
     )
     (path "/00000000-0000-0000-0000-0000617e6d54"
-      (reference "R23") (unit 1) (value "100k") (footprint "Resistor_SMD:R_0805_2012Metric")
+      (reference "R23") (unit 1) (value "100k") (footprint "Resistor_SMD:R_0603_1608Metric")
     )
     (path "/00000000-0000-0000-0000-00006078c669/00000000-0000-0000-0000-000060e2ee98"

Commit message: CC detect trigger + inner layer routing
Other:
- sheet Control ports: added PU_CC, PU_CC_1, PU_CC_2; removed none
- sheet USB 2.0 and Misc Signal Switching ports: added PU_CC, PU_CC_1, PU_CC_2; removed none

Commit message: 6 layer re-routing
Connections:
- net Control/D_N_uC renamed Control/D_uC_N
- net Control/D_P_uC renamed Control/D_uC_P
Other:
- sheet Control ports: added D_uC_N, D_uC_P; removed D_N_uC, D_P_uC
Changed lines of the file:
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@@
       (effects (font (size 1.27 1.27)) (justify right))
     )
-    (pin "D_P_uC" output (at 104.14 172.72 180)
-      (effects (font (size 1.27 1.27)) (justify left))
-    )
-    (pin "D_N_uC" output (at 104.14 175.26 180)
+    (pin "D_uC_P" output (at 104.14 172.72 180)
+      (effects (font (size 1.27 1.27)) (justify left))
+    )
+    (pin "D_uC_N" output (at 104.14 175.26 180)
       (effects (font (size 1.27 1.27)) (justify left))
     )
@@
       (reference "#PWR05") (unit 1) (value "GND") (footprint "")
     )
+    (path "/00000000-0000-0000-0000-00006086b3f3/35dca088-b88f-4e6d-bf2f-61d34196ddae"
+      (reference "#PWR06") (unit 1) (value "GND") (footprint "")
+    )
     (path "/00000000-0000-0000-0000-0000610e53f5/00000000-0000-0000-0000-00006191a7de"
       (reference "#PWR07") (unit 1) (value "GND") (footprint "")
@@
       (reference "#PWR08") (unit 1) (value "GND") (footprint "")
     )
+    (path "/00000000-0000-0000-0000-00006086b3f3/4cfa5d23-28d3-4496-88f9-e8f971816ab0"
+      (reference "#PWR09") (unit 1) (value "GND") (footprint "")
+    )
     (path "/00000000-0000-0000-0000-00006086b3f3/00000000-0000-0000-0000-000060e815b8"
       (reference "#PWR010") (unit 1) (value "GND") (footprint "")
@@
       (reference "#PWR024") (unit 1) (value "+3.3V") (footprint "")
     )
+    (path "/00000000-0000-0000-0000-00006086b3f3/d93da42e-33d0-41f7-80b6-260bceb6f799"
+      (reference "#PWR025") (unit 1) (value "GND") (footprint "")
+    )
     (path "/00000000-0000-0000-0000-00006086b3f3/00000000-0000-0000-0000-00006156ae36"
       (reference "#PWR028") (unit 1) (value "GND") (footprint "")
@@
       (reference "R28") (unit 1) (value "220k") (footprint "Resistor_SMD:R_0402_1005Metric")
     )
+    (path "/00000000-0000-0000-0000-00006086b3f3/7e95abd5-3dc5-47c3-92eb-e332a06585c6"
+      (reference "R29") (unit 1) (value "220k") (footprint "Resistor_SMD:R_0603_1608Metric")
+    )
+    (path "/00000000-0000-0000-0000-00006086b3f3/7c63d664-6d23-4b23-853b-a56c3ba17cb5"
+      (reference "R30") (unit 1) (value "220k") (footprint "Resistor_SMD:R_0603_1608Metric")
+    )
+    (path "/00000000-0000-0000-0000-00006086b3f3/248654c3-6fc0-4657-98b2-9186fcce2b8f"
+      (reference "R31") (unit 1) (value "220k") (footprint "Resistor_SMD:R_0603_1608Metric")
+    )
     (path "/00000000-0000-0000-0000-00006078c669/00000000-0000-0000-0000-000060e2ee98"

Commit message: resistor value + stitching vias
Changed lines of the file:
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@@
       (effects (font (size 1.27 1.27)) (justify left))
     )
-    (pin "PU_CC" input (at 104.14 180.34 180)
+    (pin "PU_CC" output (at 104.14 180.34 180)
       (effects (font (size 1.27 1.27)) (justify left))
     )
-    (pin "PU_CC_2" input (at 104.14 185.42 180)
+    (pin "PU_CC_2" output (at 104.14 185.42 180)
       (effects (font (size 1.27 1.27)) (justify left))
     )
-    (pin "PU_CC_1" input (at 104.14 182.88 180)
+    (pin "PU_CC_1" output (at 104.14 182.88 180)
       (effects (font (size 1.27 1.27)) (justify left))
     )
@@
     )
     (path "/00000000-0000-0000-0000-0000610e53f5/6d21c2a1-b663-4221-aad5-1393d1f17314"
-      (reference "D7") (unit 1) (value "3.3V") (footprint "Diode_SMD:D_SOD-523")
+      (reference "D7") (unit 1) (value "3.6V") (footprint "Diode_SMD:D_SOD-523")
     )
     (path "/00000000-0000-0000-0000-0000610e53f5/f74d4f11-39e8-4a3d-b4b8-25e026f99cda"
-      (reference "D8") (unit 1) (value "3.3V") (footprint "Diode_SMD:D_SOD-523")
+      (reference "D8") (unit 1) (value "3.6V") (footprint "Diode_SMD:D_SOD-523")
     )
     (path "/00000000-0000-0000-0000-0000610e53f5/86148fb1-c94e-4cc9-bf8c-b8687e7fd903"
-      (reference "D9") (unit 1) (value "3.3V") (footprint "Diode_SMD:D_SOD-523")
+      (reference "D9") (unit 1) (value "3.6V") (footprint "Diode_SMD:D_SOD-523")
     )
     (path "/00000000-0000-0000-0000-00006086b3f3/00000000-0000-0000-0000-000060eeb93a"
@@
     )
     (path "/00000000-0000-0000-0000-00006078c669/6dfdf56f-03fa-46a7-b952-05d4e94d5585"
-      (reference "Q1") (unit 1) (value "2N7002") (footprint "Package_DFN_QFN:Diodes_DFN1006-3")
+      (reference "Q1") (unit 1) (value "AP1606") (footprint "Package_DFN_QFN:Diodes_DFN1006-3")
     )
     (path "/00000000-0000-0000-0000-00006078c669/e63e441c-d563-4a4b-8680-4e2600adb301"
-      (reference "Q2") (unit 1) (value "2N7002") (footprint "Package_DFN_QFN:Diodes_DFN1006-3")
+      (reference "Q2") (unit 1) (value "AP1606") (footprint "Package_DFN_QFN:Diodes_DFN1006-3")
     )
     (path "/00000000-0000-0000-0000-00006078c669/795ef6a8-c75e-4cca-a90b-0924912a634e"
-      (reference "Q3") (unit 1) (value "2N7002") (footprint "Package_DFN_QFN:Diodes_DFN1006-3")
+      (reference "Q3") (unit 1) (value "AP1606") (footprint "Package_DFN_QFN:Diodes_DFN1006-3")
     )
     (path "/00000000-0000-0000-0000-00006078c669/cce6deed-ac7e-4607-b866-bfbff4da103b"
-      (reference "Q4") (unit 1) (value "2N7002") (footprint "Package_DFN_QFN:Diodes_DFN1006-3")
+      (reference "Q4") (unit 1) (value "AP1606") (footprint "Package_DFN_QFN:Diodes_DFN1006-3")
     )
     (path "/00000000-0000-0000-0000-00006078c669/20ce3f31-9924-4c6b-ab6b-33294af49b8b"
-      (reference "Q5") (unit 1) (value "2N7002") (footprint "Package_DFN_QFN:Diodes_DFN1006-3")
+      (reference "Q5") (unit 1) (value "AP1606") (footprint "Package_DFN_QFN:Diodes_DFN1006-3")
     )
     (path "/00000000-0000-0000-0000-00006078c669/e3c91051-0b41-4302-b163-038ad51c80b2"
-      (reference "Q6") (unit 1) (value "2N7002") (footprint "Package_DFN_QFN:Diodes_DFN1006-3")
+      (reference "Q6") (unit 1) (value "AP1606") (footprint "Package_DFN_QFN:Diodes_DFN1006-3")
     )
     (path "/00000000-0000-0000-0000-0000610e53f5/00000000-0000-0000-0000-000060142a37"
-      (reference "R1") (unit 1) (value "220") (footprint "Resistor_SMD:R_0603_1608Metric")
+      (reference "R1") (unit 1) (value "470") (footprint "Resistor_SMD:R_0603_1608Metric")
     )
     (path "/00000000-0000-0000-0000-0000610e53f5/00000000-0000-0000-0000-000060140919"
-      (reference "R2") (unit 1) (value "220") (footprint "Resistor_SMD:R_0603_1608Metric")
+      (reference "R2") (unit 1) (value "470") (footprint "Resistor_SMD:R_0603_1608Metric")
     )
     (path "/00000000-0000-0000-0000-0000610e53f5/00000000-0000-0000-0000-0000616a374f"
-      (reference "R3") (unit 1) (value "220") (footprint "Resistor_SMD:R_0603_1608Metric")
+      (reference "R3") (unit 1) (value "470") (footprint "Resistor_SMD:R_0603_1608Metric")
     )
     (path "/00000000-0000-0000-0000-00006086b3f3/00000000-0000-0000-0000-0000600bbec3"
-      (reference "R4") (unit 1) (value "9k") (footprint "Resistor_SMD:R_0603_1608Metric")
+      (reference "R4") (unit 1) (value "10k") (footprint "Resistor_SMD:R_0603_1608Metric")
     )
     (path "/00000000-0000-0000-0000-00006086b3f3/00000000-0000-0000-0000-0000600c3d30"
-      (reference "R5") (unit 1) (value "9k") (footprint "Resistor_SMD:R_0603_1608Metric")
+      (reference "R5") (unit 1) (value "10k") (footprint "Resistor_SMD:R_0603_1608Metric")
     )
     (path "/00000000-0000-0000-0000-00006060e5e3/00000000-0000-0000-0000-00006012d6cb"
@@
     )
     (path "/00000000-0000-0000-0000-00006086b3f3/00000000-0000-0000-0000-00006156ae26"
-      (reference "R13") (unit 1) (value "9k") (footprint "Resistor_SMD:R_0603_1608Metric")
+      (reference "R13") (unit 1) (value "47k") (footprint "Resistor_SMD:R_0603_1608Metric")
     )
     (path "/00000000-0000-0000-0000-00006086b3f3/00000000-0000-0000-0000-00006156ae2c"
-      (reference "R14") (unit 1) (value "1k") (footprint "Resistor_SMD:R_0603_1608Metric")
+      (reference "R14") (unit 1) (value "5.6k") (footprint "Resistor_SMD:R_0603_1608Metric")
     )
     (path "/00000000-0000-0000-0000-00006086b3f3/00000000-0000-0000-0000-0000615833ba"
-      (reference "R15") (unit 1) (value "9k") (footprint "Resistor_SMD:R_0603_1608Metric")
+      (reference "R15") (unit 1) (value "47k") (footprint "Resistor_SMD:R_0603_1608Metric")
     )
     (path "/00000000-0000-0000-0000-00006086b3f3/00000000-0000-0000-0000-0000615833c0"
-      (reference "R16") (unit 1) (value "1k") (footprint "Resistor_SMD:R_0603_1608Metric")
+      (reference "R16") (unit 1) (value "5.6k") (footprint "Resistor_SMD:R_0603_1608Metric")
     )
     (path "/00000000-0000-0000-0000-00006086b3f3/00000000-0000-0000-0000-00006158fd1f"
-      (reference "R17") (unit 1) (value "9k") (footprint "Resistor_SMD:R_0603_1608Metric")
+      (reference "R17") (unit 1) (value "47k") (footprint "Resistor_SMD:R_0603_1608Metric")
     )
     (path "/00000000-0000-0000-0000-00006086b3f3/00000000-0000-0000-0000-00006158fd25"
-      (reference "R18") (unit 1) (value "1k") (footprint "Resistor_SMD:R_0603_1608Metric")
+      (reference "R18") (unit 1) (value "5.6k") (footprint "Resistor_SMD:R_0603_1608Metric")
     )
     (path "/00000000-0000-0000-0000-0000610e53f5/00000000-0000-0000-0000-000061664e03"
