File: KiCad/h_control.kicad_sch (KiCad schematic)
At the start: 14 parts, among them J4 Conn_02x05_Odd_Even, SW1 SW_Push, U9 ATSAMD21E15B-M

Commit message: Use 0603 resistors and capacitors
Parts:
- C4, C5, C6, C7: footprint Capacitor_SMD:C_0805_2012Metric -> Capacitor_SMD:C_0603_1608Metric
- R1, R19, R2, R3: footprint Resistor_SMD:R_0805_2012Metric -> Resistor_SMD:R_0603_1608Metric
Changed lines of the file:
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@@
     (property "Reference" "R2" (id 0) (at 118.11 69.85 90))
     (property "Value" "220" (id 1) (at 125.73 69.85 90))
-    (property "Footprint" "Resistor_SMD:R_0805_2012Metric" (id 2) (at 121.92 68.58 0)
+    (property "Footprint" "Resistor_SMD:R_0603_1608Metric" (id 2) (at 121.92 68.58 0)
       (effects (font (size 1.27 1.27)) hide)
     )
@@
     (property "Reference" "R1" (id 0) (at 118.11 105.41 90))
     (property "Value" "220" (id 1) (at 125.73 105.41 90))
-    (property "Footprint" "Resistor_SMD:R_0805_2012Metric" (id 2) (at 121.92 104.14 0)
+    (property "Footprint" "Resistor_SMD:R_0603_1608Metric" (id 2) (at 121.92 104.14 0)
       (effects (font (size 1.27 1.27)) hide)
     )
@@
       (effects (font (size 1.27 1.27)) (justify left))
     )
-    (property "Footprint" "Capacitor_SMD:C_0805_2012Metric" (id 2) (at 121.92 46.99 0)
+    (property "Footprint" "Capacitor_SMD:C_0603_1608Metric" (id 2) (at 121.92 46.99 0)
       (effects (font (size 1.27 1.27)) hide)
     )
@@
       (effects (font (size 1.27 1.27)) (justify left))
     )
-    (property "Footprint" "Capacitor_SMD:C_0805_2012Metric" (id 2) (at 133.35 46.99 0)
+    (property "Footprint" "Capacitor_SMD:C_0603_1608Metric" (id 2) (at 133.35 46.99 0)
       (effects (font (size 1.27 1.27)) hide)
     )
@@
     (property "Reference" "R19" (id 0) (at 118.11 130.81 90))
     (property "Value" "1k" (id 1) (at 118.11 135.89 90))
-    (property "Footprint" "Resistor_SMD:R_0805_2012Metric" (id 2) (at 118.11 133.35 0)
+    (property "Footprint" "Resistor_SMD:R_0603_1608Metric" (id 2) (at 118.11 133.35 0)
       (effects (font (size 1.27 1.27)) hide)
     )
@@
     (property "Reference" "R3" (id 0) (at 118.11 100.33 90))
     (property "Value" "220" (id 1) (at 125.73 100.33 90))
-    (property "Footprint" "Resistor_SMD:R_0805_2012Metric" (id 2) (at 121.92 101.6 0)
+    (property "Footprint" "Resistor_SMD:R_0603_1608Metric" (id 2) (at 121.92 101.6 0)
       (effects (font (size 1.27 1.27)) hide)
     )
@@
       (effects (font (size 1.27 1.27)) (justify left))
     )
-    (property "Footprint" "Capacitor_SMD:C_0805_2012Metric" (id 2) (at 189.23 46.99 0)
+    (property "Footprint" "Capacitor_SMD:C_0603_1608Metric" (id 2) (at 189.23 46.99 0)
       (effects (font (size 1.27 1.27)) hide)
     )
@@
       (effects (font (size 1.27 1.27)) (justify left))
     )
-    (property "Footprint" "Capacitor_SMD:C_0805_2012Metric" (id 2) (at 177.8 46.99 0)
-      (effects (font (size 1.27 1.27)) hide)
-    )
+    (property "Footprint" "Capacitor_SMD:C_0603_1608Metric" (id 2) (at 177.8 46.99 0)
+      (effects (font (size 1.27 1.27)) hide)
+    )

Commit message: CC detect trigger + inner layer routing
Parts:
- added D7, D8, D9: 3.3V, Diode_SMD:D_SOD-523, symbol Diode:BZV55B3V3
Connections:
- net GND: now also D7.2 (A), D8.2 (A), D9.2 (A)
- net PU_CC_2: now reaches U9.13 (PA10)
- net PU_CC_2: now also D7.1 (K)
- net PU_CC: now reaches U9.14 (PA11)
- net PU_CC: now also D9.1 (K)
- net PU_CC_1: now reaches U9.8 (PA07)
- net PU_CC_1: now also D8.1 (K)
- no-connect marks 8 -> 5

Commit message: 6 layer re-routing
Connections:
- net D_N_uC renamed D_uC_N
- net D_P_uC renamed D_uC_P
Changed lines of the file:
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@@
     (effects (font (size 1.27 1.27)) (justify right))
   )
-  (hierarchical_label "D_N_uC" (shape input) (at 91.44 121.92 180)
+  (hierarchical_label "D_uC_N" (shape input) (at 91.44 121.92 180)
     (effects (font (size 1.27 1.27)) (justify right))
   )
@@
     (effects (font (size 1.27 1.27)) (justify right))
   )
-  (hierarchical_label "D_P_uC" (shape input) (at 91.44 124.46 180)
+  (hierarchical_label "D_uC_P" (shape input) (at 91.44 124.46 180)
     (effects (font (size 1.27 1.27)) (justify right))
   )

Commit message: resistor value + stitching vias
Parts:
- D7, D8, D9: value 3.3V -> 3.6V
- R1, R2, R3: value 220 -> 470
Changed lines of the file:
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@@
     (stroke (width 0) (type default) (color 0 0 0 0))
   )
-  (wire (pts (xy 92.71 137.16) (xy 100.33 137.16))
+  (wire (pts (xy 92.71 137.16) (xy 101.6 137.16))
     (stroke (width 0) (type default) (color 0 0 0 0))
   )
@@
     (stroke (width 0) (type default) (color 0 0 0 0))
   )
+  (wire (pts (xy 123.19 137.16) (xy 139.7 137.16))
+    (stroke (width 0) (type default) (color 0 0 0 0))
+  )
   (wire (pts (xy 177.8 43.18) (xy 165.1 43.18))
     (stroke (width 0) (type default) (color 0 0 0 0))
   )
-  (wire (pts (xy 102.87 137.16) (xy 102.87 139.7))
+  (wire (pts (xy 103.505 137.16) (xy 101.6 139.7))
     (stroke (width 0) (type default) (color 0 0 0 0))
   )
@@
     (stroke (width 0) (type default) (color 0 0 0 0))
   )
-  (wire (pts (xy 105.41 139.7) (xy 139.7 139.7))
-    (stroke (width 0) (type default) (color 0 0 0 0))
-  )
   (wire (pts (xy 115.57 133.35) (xy 76.2 133.35))
     (stroke (width 0) (type default) (color 0 0 0 0))
@@
     (stroke (width 0) (type default) (color 0 0 0 0))
   )
+  (wire (pts (xy 103.505 139.7) (xy 139.7 139.7))
+    (stroke (width 0) (type default) (color 0 0 0 0))
+  )
   (wire (pts (xy 189.23 49.53) (xy 189.23 50.8))
     (stroke (width 0) (type default) (color 0 0 0 0))
@@
     (stroke (width 0) (type default) (color 0 0 0 0))
   )
-  (wire (pts (xy 105.41 139.7) (xy 105.41 135.89))
-    (stroke (width 0) (type default) (color 0 0 0 0))
-  )
-  (wire (pts (xy 123.19 137.16) (xy 139.7 137.16))
+  (wire (pts (xy 103.505 139.7) (xy 101.6 137.16))
     (stroke (width 0) (type default) (color 0 0 0 0))
   )
@@
     (stroke (width 0) (type default) (color 0 0 0 0))
   )
+  (wire (pts (xy 123.19 137.16) (xy 103.505 137.16))
+    (stroke (width 0) (type default) (color 0 0 0 0))
+  )
   (wire (pts (xy 91.44 81.28) (xy 139.7 81.28))
     (stroke (width 0) (type default) (color 0 0 0 0))
@@
     (stroke (width 0) (type default) (color 0 0 0 0))
   )
-  (wire (pts (xy 92.71 139.7) (xy 102.87 139.7))
+  (wire (pts (xy 92.71 139.7) (xy 101.6 139.7))
     (stroke (width 0) (type default) (color 0 0 0 0))
   )
@@
     (stroke (width 0) (type default) (color 0 0 0 0))
   )
-  (wire (pts (xy 123.19 137.16) (xy 102.87 137.16))
-    (stroke (width 0) (type default) (color 0 0 0 0))
-  )
   (wire (pts (xy 121.92 43.18) (xy 121.92 44.45))
     (stroke (width 0) (type default) (color 0 0 0 0))
   )
-  (wire (pts (xy 100.33 135.89) (xy 100.33 137.16))
-    (stroke (width 0) (type default) (color 0 0 0 0))
-  )
   (wire (pts (xy 80.01 147.32) (xy 76.2 147.32))
     (stroke (width 0) (type default) (color 0 0 0 0))
@@
   )
   (wire (pts (xy 182.88 50.8) (xy 177.8 50.8))
-    (stroke (width 0) (type default) (color 0 0 0 0))
-  )
-  (wire (pts (xy 105.41 135.89) (xy 100.33 135.89))
     (stroke (width 0) (type default) (color 0 0 0 0))
   )
@@
     (effects (font (size 1.27 1.27)) (justify right))
   )
-  (hierarchical_label "PU_CC" (shape input) (at 55.245 88.9 180)
+  (hierarchical_label "PU_CC" (shape output) (at 55.245 88.9 180)
     (effects (font (size 1.27 1.27)) (justify right))
   )
@@
     (effects (font (size 1.27 1.27)) (justify right))
   )
-  (hierarchical_label "PU_CC_1" (shape input) (at 55.245 78.74 180)
+  (hierarchical_label "PU_CC_1" (shape output) (at 55.245 78.74 180)
     (effects (font (size 1.27 1.27)) (justify right))
   )
@@
     (effects (font (size 1.27 1.27)) (justify right))
   )
-  (hierarchical_label "PU_CC_2" (shape input) (at 55.245 86.36 180)
+  (hierarchical_label "PU_CC_2" (shape output) (at 55.245 86.36 180)
     (effects (font (size 1.27 1.27)) (justify right))
   )
@@
     (in_bom yes) (on_board yes)
     (property "Reference" "R2" (id 0) (at 118.11 69.85 90))
-    (property "Value" "220" (id 1) (at 125.73 69.85 90))
+    (property "Value" "470" (id 1) (at 125.73 69.85 90))
     (property "Footprint" "Resistor_SMD:R_0603_1608Metric" (id 2) (at 121.92 68.58 0)
       (effects (font (size 1.27 1.27)) hide)
@@
     (in_bom yes) (on_board yes)
     (property "Reference" "R1" (id 0) (at 118.11 105.41 90))
-    (property "Value" "220" (id 1) (at 125.73 105.41 90))
+    (property "Value" "470" (id 1) (at 125.73 105.41 90))
     (property "Footprint" "Resistor_SMD:R_0603_1608Metric" (id 2) (at 121.92 104.14 0)
       (effects (font (size 1.27 1.27)) hide)
@@
     (in_bom yes) (on_board yes)
     (property "Reference" "R3" (id 0) (at 118.11 100.33 90))
-    (property "Value" "220" (id 1) (at 125.73 100.33 90))
+    (property "Value" "470" (id 1) (at 125.73 100.33 90))
     (property "Footprint" "Resistor_SMD:R_0603_1608Metric" (id 2) (at 121.92 101.6 0)
       (effects (font (size 1.27 1.27)) hide)
@@
       (effects (font (size 1.27 1.27)) (justify left))
     )
-    (property "Value" "3.3V" (id 1) (at 60.96 93.98 90)
+    (property "Value" "3.6V" (id 1) (at 60.96 93.98 90)
       (effects (font (size 1.27 1.27)) (justify left))
     )
@@
       (effects (font (size 1.27 1.27)) (justify left))
     )
-    (property "Value" "3.3V" (id 1) (at 68.58 96.52 90)
+    (property "Value" "3.6V" (id 1) (at 68.58 96.52 90)
       (effects (font (size 1.27 1.27)) (justify left))
     )
@@
       (effects (font (size 1.27 1.27)) (justify left))
     )
-    (property "Value" "3.3V" (id 1) (at 73.66 83.185 0)
-      (effects (font (size 1.27 1.27)) (justify left))
-    )
+    (property "Value" "3.6V" (id 1) (at 73.66 83.185 0)
+      (effects (font (size 1.27 1.27)) (justify left))
+    )
