File: KiCad/h_power.kicad_sch (KiCad schematic)
At the start: 27 parts, among them U4 AP63205WU, U5 UCS3205-E_Q8A, U6 UCS3205-E_Q8A, U8 AZ1117C-3.3

Commit message: Use 0603 resistors and capacitors
Parts:
- C1: footprint Capacitor_SMD:C_0805_2012Metric -> Capacitor_SMD:C_0603_1608Metric
- R10, R13, R14, R15, R16, R17, R18, R4, R5, R9: footprint Resistor_SMD:R_0805_2012Metric -> Resistor_SMD:R_0603_1608Metric
Changed lines of the file:
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@@
       (effects (font (size 1.27 1.27)) (justify right))
     )
-    (property "Footprint" "Resistor_SMD:R_0805_2012Metric" (id 2) (at 101.6 46.99 0)
+    (property "Footprint" "Resistor_SMD:R_0603_1608Metric" (id 2) (at 101.6 46.99 0)
       (effects (font (size 1.27 1.27)) hide)
     )
@@
       (effects (font (size 1.27 1.27)) (justify right))
     )
-    (property "Footprint" "Resistor_SMD:R_0805_2012Metric" (id 2) (at 102.87 96.52 0)
+    (property "Footprint" "Resistor_SMD:R_0603_1608Metric" (id 2) (at 102.87 96.52 0)
       (effects (font (size 1.27 1.27)) hide)
     )
@@
       (effects (font (size 1.27 1.27)) (justify left))
     )
-    (property "Footprint" "Resistor_SMD:R_0805_2012Metric" (id 2) (at 185.42 62.23 0)
+    (property "Footprint" "Resistor_SMD:R_0603_1608Metric" (id 2) (at 185.42 62.23 0)
       (effects (font (size 1.27 1.27)) hide)
     )
@@
       (effects (font (size 1.27 1.27)) (justify left))
     )
-    (property "Footprint" "Resistor_SMD:R_0805_2012Metric" (id 2) (at 185.42 111.76 0)
+    (property "Footprint" "Resistor_SMD:R_0603_1608Metric" (id 2) (at 185.42 111.76 0)
       (effects (font (size 1.27 1.27)) hide)
     )
@@
       (effects (font (size 1.27 1.27)) (justify left))
     )
-    (property "Footprint" "Capacitor_SMD:C_0805_2012Metric" (id 2) (at 140.97 143.51 0)
+    (property "Footprint" "Capacitor_SMD:C_0603_1608Metric" (id 2) (at 140.97 143.51 0)
       (effects (font (size 1.27 1.27)) hide)
     )
@@
       (effects (font (size 1.27 1.27)) (justify right))
     )
-    (property "Footprint" "Resistor_SMD:R_0805_2012Metric" (id 2) (at 69.85 171.45 0)
+    (property "Footprint" "Resistor_SMD:R_0603_1608Metric" (id 2) (at 69.85 171.45 0)
       (effects (font (size 1.27 1.27)) hide)
     )
@@
       (effects (font (size 1.27 1.27)) (justify right))
     )
-    (property "Footprint" "Resistor_SMD:R_0805_2012Metric" (id 2) (at 69.85 181.61 0)
+    (property "Footprint" "Resistor_SMD:R_0603_1608Metric" (id 2) (at 69.85 181.61 0)
       (effects (font (size 1.27 1.27)) hide)
     )
@@
       (effects (font (size 1.27 1.27)) (justify right))
     )
-    (property "Footprint" "Resistor_SMD:R_0805_2012Metric" (id 2) (at 109.22 172.72 0)
+    (property "Footprint" "Resistor_SMD:R_0603_1608Metric" (id 2) (at 109.22 172.72 0)
       (effects (font (size 1.27 1.27)) hide)
     )
@@
       (effects (font (size 1.27 1.27)) (justify right))
     )
-    (property "Footprint" "Resistor_SMD:R_0805_2012Metric" (id 2) (at 109.22 182.88 0)
+    (property "Footprint" "Resistor_SMD:R_0603_1608Metric" (id 2) (at 109.22 182.88 0)
       (effects (font (size 1.27 1.27)) hide)
     )
@@
       (effects (font (size 1.27 1.27)) (justify right))
     )
-    (property "Footprint" "Resistor_SMD:R_0805_2012Metric" (id 2) (at 140.97 172.72 0)
+    (property "Footprint" "Resistor_SMD:R_0603_1608Metric" (id 2) (at 140.97 172.72 0)
       (effects (font (size 1.27 1.27)) hide)
     )
@@
       (effects (font (size 1.27 1.27)) (justify right))
     )
-    (property "Footprint" "Resistor_SMD:R_0805_2012Metric" (id 2) (at 140.97 182.88 0)
-      (effects (font (size 1.27 1.27)) hide)
-    )
+    (property "Footprint" "Resistor_SMD:R_0603_1608Metric" (id 2) (at 140.97 182.88 0)
+      (effects (font (size 1.27 1.27)) hide)
+    )

Commit message: 6 layer re-routing
Parts:
- added R29, R30, R31: 220k, Resistor_SMD:R_0603_1608Metric, symbol Device:R_Small
Connections:
- net GND: now also R29.1, R30.1, R31.1
- net VBUS_IN1_FUSED: now also R29.2
- net VBUS_IN2_FUSED: now also R30.2
- net VBUS_OUT_FUSED: now also R31.2
Changed lines of the file:
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@@
   (junction (at 165.1 139.7) (diameter 0) (color 0 0 0 0)
   )
+  (junction (at 126.365 160.02) (diameter 0) (color 0 0 0 0)
+  )
   (junction (at 203.2 139.7) (diameter 0) (color 0 0 0 0)
   )
+  (junction (at 95.885 165.1) (diameter 0) (color 0 0 0 0)
+  )
   (junction (at 125.73 88.9) (diameter 0) (color 0 0 0 0)
   )
@@
   )
   (junction (at 69.85 176.53) (diameter 0) (color 0 0 0 0)
+  )
+  (junction (at 69.85 163.195) (diameter 0) (color 0 0 0 0)
   )
   (junction (at 81.28 69.85) (diameter 0) (color 0 0 0 0)
@@
   (no_connect (at 173.99 64.77))
   (no_connect (at 173.99 114.3))
+  (wire (pts (xy 58.42 163.195) (xy 69.85 163.195))
+    (stroke (width 0) (type default) (color 0 0 0 0))
+  )
   (wire (pts (xy 115.57 177.8) (xy 109.22 177.8))
     (stroke (width 0) (type default) (color 0 0 0 0))
@@
     (stroke (width 0) (type default) (color 0 0 0 0))
   )
+  (wire (pts (xy 126.365 167.005) (xy 126.365 168.275))
+    (stroke (width 0) (type default) (color 0 0 0 0))
+  )
   (wire (pts (xy 125.73 44.45) (xy 133.35 44.45))
     (stroke (width 0) (type default) (color 0 0 0 0))
@@
     (stroke (width 0) (type default) (color 0 0 0 0))
   )
+  (wire (pts (xy 58.42 163.195) (xy 58.42 171.45))
+    (stroke (width 0) (type default) (color 0 0 0 0))
+  )
   (wire (pts (xy 140.97 185.42) (xy 140.97 187.96))
     (stroke (width 0) (type default) (color 0 0 0 0))
@@
     (stroke (width 0) (type default) (color 0 0 0 0))
   )
+  (wire (pts (xy 69.85 163.195) (xy 69.85 168.91))
+    (stroke (width 0) (type default) (color 0 0 0 0))
+  )
   (wire (pts (xy 101.6 50.8) (xy 109.22 50.8))
     (stroke (width 0) (type default) (color 0 0 0 0))
@@
     (stroke (width 0) (type default) (color 0 0 0 0))
   )
+  (wire (pts (xy 126.365 160.02) (xy 140.97 160.02))
+    (stroke (width 0) (type default) (color 0 0 0 0))
+  )
   (wire (pts (xy 176.53 46.99) (xy 173.99 46.99))
     (stroke (width 0) (type default) (color 0 0 0 0))
@@
     (stroke (width 0) (type default) (color 0 0 0 0))
   )
+  (wire (pts (xy 95.885 165.1) (xy 95.885 167.005))
+    (stroke (width 0) (type default) (color 0 0 0 0))
+  )
   (wire (pts (xy 179.07 39.37) (xy 179.07 49.53))
     (stroke (width 0) (type default) (color 0 0 0 0))
@@
     (stroke (width 0) (type default) (color 0 0 0 0))
   )
+  (wire (pts (xy 95.885 165.1) (xy 109.22 165.1))
+    (stroke (width 0) (type default) (color 0 0 0 0))
+  )
   (wire (pts (xy 173.99 104.14) (xy 195.58 104.14))
     (stroke (width 0) (type default) (color 0 0 0 0))
@@
     (stroke (width 0) (type default) (color 0 0 0 0))
   )
-  (wire (pts (xy 73.66 165.1) (xy 109.22 165.1))
+  (wire (pts (xy 73.66 165.1) (xy 95.885 165.1))
     (stroke (width 0) (type default) (color 0 0 0 0))
   )
@@
     (stroke (width 0) (type default) (color 0 0 0 0))
   )
-  (wire (pts (xy 69.85 139.7) (xy 69.85 168.91))
+  (wire (pts (xy 69.85 139.7) (xy 69.85 163.195))
     (stroke (width 0) (type default) (color 0 0 0 0))
   )
@@
     (stroke (width 0) (type default) (color 0 0 0 0))
   )
+  (wire (pts (xy 95.885 172.085) (xy 95.885 173.355))
+    (stroke (width 0) (type default) (color 0 0 0 0))
+  )
   (wire (pts (xy 201.93 81.28) (xy 201.93 87.63))
     (stroke (width 0) (type default) (color 0 0 0 0))
@@
     (stroke (width 0) (type default) (color 0 0 0 0))
   )
+  (wire (pts (xy 58.42 176.53) (xy 58.42 177.8))
+    (stroke (width 0) (type default) (color 0 0 0 0))
+  )
   (wire (pts (xy 101.6 49.53) (xy 101.6 50.8))
     (stroke (width 0) (type default) (color 0 0 0 0))
@@
     (stroke (width 0) (type default) (color 0 0 0 0))
   )
-  (wire (pts (xy 77.47 160.02) (xy 140.97 160.02))
+  (wire (pts (xy 77.47 160.02) (xy 126.365 160.02))
     (stroke (width 0) (type default) (color 0 0 0 0))
   )
   (wire (pts (xy 195.58 67.31) (xy 195.58 68.58))
+    (stroke (width 0) (type default) (color 0 0 0 0))
+  )
+  (wire (pts (xy 126.365 160.02) (xy 126.365 161.925))
     (stroke (width 0) (type default) (color 0 0 0 0))
   )
@@
     (pin "3")
   )
+  (symbol (lib_id "Device:R_Small") (at 126.365 164.465 0) (mirror x) (unit 1)
+    (in_bom yes) (on_board yes)
+    (property "Reference" "R31" (id 0) (at 124.8918 163.2966 0)
+      (effects (font (size 1.27 1.27)) (justify right))
+    )
+    (property "Value" "220k" (id 1) (at 124.8918 165.608 0)
+      (effects (font (size 1.27 1.27)) (justify right))
+    )
+    (property "Footprint" "Resistor_SMD:R_0603_1608Metric" (id 2) (at 126.365 164.465 0)
+      (effects (font (size 1.27 1.27)) hide)
+    )
+    (property "Datasheet" "~" (id 3) (at 126.365 164.465 0)
+      (effects (font (size 1.27 1.27)) hide)
+    )
+    (pin "1")
+    (pin "2")
+  )
+  (symbol (lib_id "power:GND") (at 58.42 177.8 0) (unit 1)
+    (in_bom yes) (on_board yes)
+    (property "Reference" "#PWR06" (id 0) (at 58.42 184.15 0)
+      (effects (font (size 1.27 1.27)) hide)
+    )
+    (property "Value" "GND" (id 1) (at 58.547 182.1942 0))
+    (property "Footprint" "" (id 2) (at 58.42 177.8 0)
+      (effects (font (size 1.27 1.27)) hide)
+    )
+    (property "Datasheet" "" (id 3) (at 58.42 177.8 0)
+      (effects (font (size 1.27 1.27)) hide)
+    )
+    (pin "1")
+  )
+  (symbol (lib_id "power:GND") (at 95.885 173.355 0) (unit 1)
+    (in_bom yes) (on_board yes)
+    (property "Reference" "#PWR09" (id 0) (at 95.885 179.705 0)
+      (effects (font (size 1.27 1.27)) hide)
+    )
+    (property "Value" "GND" (id 1) (at 96.012 177.7492 0))
+    (property "Footprint" "" (id 2) (at 95.885 173.355 0)
+      (effects (font (size 1.27 1.27)) hide)
+    )
+    (property "Datasheet" "" (id 3) (at 95.885 173.355 0)
+      (effects (font (size 1.27 1.27)) hide)
+    )
+    (pin "1")
+  )
+  (symbol (lib_id "Device:R_Small") (at 95.885 169.545 0) (mirror x) (unit 1)
+    (in_bom yes) (on_board yes)
+    (property "Reference" "R30" (id 0) (at 94.4118 168.3766 0)
+      (effects (font (size 1.27 1.27)) (justify right))
+    )
+    (property "Value" "220k" (id 1) (at 94.4118 170.688 0)
+      (effects (font (size 1.27 1.27)) (justify right))
+    )
+    (property "Footprint" "Resistor_SMD:R_0603_1608Metric" (id 2) (at 95.885 169.545 0)
+      (effects (font (size 1.27 1.27)) hide)
+    )
+    (property "Datasheet" "~" (id 3) (at 95.885 169.545 0)
+      (effects (font (size 1.27 1.27)) hide)
+    )
+    (pin "1")
+    (pin "2")
+  )
+  (symbol (lib_id "Device:R_Small") (at 58.42 173.99 0) (mirror x) (unit 1)
+    (in_bom yes) (on_board yes)
+    (property "Reference" "R29" (id 0) (at 56.9468 172.8216 0)
+      (effects (font (size 1.27 1.27)) (justify right))
+    )
+    (property "Value" "220k" (id 1) (at 56.9468 175.133 0)
+      (effects (font (size 1.27 1.27)) (justify right))
+    )
+    (property "Footprint" "Resistor_SMD:R_0603_1608Metric" (id 2) (at 58.42 173.99 0)
+      (effects (font (size 1.27 1.27)) hide)
+    )
+    (property "Datasheet" "~" (id 3) (at 58.42 173.99 0)
+      (effects (font (size 1.27 1.27)) hide)
+    )
+    (pin "1")
+    (pin "2")
+  )
+  (symbol (lib_id "power:GND") (at 126.365 168.275 0) (unit 1)
+    (in_bom yes) (on_board yes)
+    (property "Reference" "#PWR025" (id 0) (at 126.365 174.625 0)
+      (effects (font (size 1.27 1.27)) hide)
+    )
+    (property "Value" "GND" (id 1) (at 126.492 172.6692 0))
+    (property "Footprint" "" (id 2) (at 126.365 168.275 0)
+      (effects (font (size 1.27 1.27)) hide)
+    )
+    (property "Datasheet" "" (id 3) (at 126.365 168.275 0)
+      (effects (font (size 1.27 1.27)) hide)
+    )
+    (pin "1")
+  )
 )

Commit message: resistor value + stitching vias
Parts:
- R13, R15, R17: value 9k -> 47k
- R14, R16, R18: value 1k -> 5.6k
- R4, R5: value 9k -> 10k
Changed lines of the file:
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@@
       (effects (font (size 1.27 1.27)) (justify right))
     )
-    (property "Value" "9k" (id 1) (at 100.1268 48.133 0)
+    (property "Value" "10k" (id 1) (at 100.1268 48.133 0)
       (effects (font (size 1.27 1.27)) (justify right))
     )
@@
       (effects (font (size 1.27 1.27)) (justify right))
     )
-    (property "Value" "9k" (id 1) (at 101.3968 97.663 0)
+    (property "Value" "10k" (id 1) (at 101.3968 97.663 0)
       (effects (font (size 1.27 1.27)) (justify right))
     )
@@
       (effects (font (size 1.27 1.27)) (justify right))
     )
-    (property "Value" "9k" (id 1) (at 68.3768 172.593 0)
+    (property "Value" "47k" (id 1) (at 68.3768 172.593 0)
       (effects (font (size 1.27 1.27)) (justify right))
     )
@@
       (effects (font (size 1.27 1.27)) (justify right))
     )
-    (property "Value" "1k" (id 1) (at 68.3768 182.753 0)
+    (property "Value" "5.6k" (id 1) (at 68.3768 182.753 0)
       (effects (font (size 1.27 1.27)) (justify right))
     )
@@
       (effects (font (size 1.27 1.27)) (justify right))
     )
-    (property "Value" "9k" (id 1) (at 107.7468 173.863 0)
+    (property "Value" "47k" (id 1) (at 107.7468 173.863 0)
       (effects (font (size 1.27 1.27)) (justify right))
     )
@@
       (effects (font (size 1.27 1.27)) (justify right))
     )
-    (property "Value" "1k" (id 1) (at 107.7468 184.023 0)
+    (property "Value" "5.6k" (id 1) (at 107.7468 184.023 0)
       (effects (font (size 1.27 1.27)) (justify right))
     )
@@
       (effects (font (size 1.27 1.27)) (justify right))
     )
-    (property "Value" "9k" (id 1) (at 139.4968 173.863 0)
+    (property "Value" "47k" (id 1) (at 139.4968 173.863 0)
       (effects (font (size 1.27 1.27)) (justify right))
     )
@@
       (effects (font (size 1.27 1.27)) (justify right))
     )
-    (property "Value" "1k" (id 1) (at 139.4968 184.023 0)
-      (effects (font (size 1.27 1.27)) (justify right))
-    )
+    (property "Value" "5.6k" (id 1) (at 139.4968 184.023 0)
+      (effects (font (size 1.27 1.27)) (justify right))
+    )
