File: KiCad/h_usb2_misc.kicad_sch (KiCad schematic)
At the start: 3 parts, among them U3 NL3S588, U7 NL3S588

Commit message: CC detect trigger + inner layer routing
Parts:
- added Q1, Q2, Q3, Q4, Q5, Q6: 2N7002, Package_DFN_QFN:Diodes_DFN1006-3, symbol Transistor_FET:2N7002
- added R11, R12, R22, R24, R25, R26: 5.1k, Resistor_SMD:R_0402_1005Metric, symbol Device:R_Small
- added R20, R21, R27, R28, R7, R8: 220k, Resistor_SMD:R_0402_1005Metric, symbol Device:R_Small
Connections:
- net CC1: now also R26.1, R28.1
- net CC1_1: now also R12.1, R8.1
- net CC1_2: now also R11.1, R7.1
- net CC2: now also R22.1, R27.1
- net CC2_1: now also R21.1, R25.1
- net CC2_2: now also R20.1, R24.1
- net GND: now also Q1.2 (S), Q2.2 (S), Q3.2 (S), Q4.2 (S), Q5.2 (S), Q6.2 (S)
- new net: Q4.3 (D), R24.2
- new net: Q3.3 (D), R22.2
- new net: Q5.3 (D), R25.2
- new net: Q6.3 (D), R26.2
- new net: Q1.3 (D), R11.2
- new net: Q2.3 (D), R12.2
- new net PU_CC: Q3.1 (G), Q6.1 (G), R27.2, R28.2
- new net PU_CC_1: Q2.1 (G), Q5.1 (G), R21.2, R8.2
- new net PU_CC_2: Q1.1 (G), Q4.1 (G), R20.2, R7.2

Commit message: resistor value + stitching vias
Parts:
- Q1, Q2, Q3, Q4, Q5, Q6: value 2N7002 -> AP1606
Changed lines of the file:
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@@
   (symbol (lib_id "Device:R_Small") (at 67.31 152.4 0) (unit 1)
     (in_bom yes) (on_board yes)
-    (property "Reference" "R24" (id 0) (at 69.85 153.035 0))
-    (property "Value" "5.1k" (id 1) (at 70.485 151.13 0))
+    (property "Reference" "R24" (id 0) (at 70.485 151.13 0))
+    (property "Value" "5.1k" (id 1) (at 70.485 153.67 0))
     (property "Footprint" "Resistor_SMD:R_0402_1005Metric" (id 2) (at 67.31 152.4 0)
       (effects (font (size 1.27 1.27)) hide)
@@
   (symbol (lib_id "Device:R_Small") (at 181.61 132.08 0) (mirror y) (unit 1)
     (in_bom yes) (on_board yes)
-    (property "Reference" "R22" (id 0) (at 179.07 132.715 0))
-    (property "Value" "5.1k" (id 1) (at 178.435 130.81 0))
+    (property "Reference" "R22" (id 0) (at 177.8 130.81 0))
+    (property "Value" "5.1k" (id 1) (at 177.8 133.35 0))
     (property "Footprint" "Resistor_SMD:R_0402_1005Metric" (id 2) (at 181.61 132.08 0)
       (effects (font (size 1.27 1.27)) hide)
@@
   (symbol (lib_id "Device:R_Small") (at 58.42 152.4 0) (unit 1)
     (in_bom yes) (on_board yes)
-    (property "Reference" "R20" (id 0) (at 60.96 153.035 0))
-    (property "Value" "220k" (id 1) (at 61.595 151.13 0))
+    (property "Reference" "R20" (id 0) (at 61.595 151.13 0))
+    (property "Value" "220k" (id 1) (at 62.23 153.67 0))
     (property "Footprint" "Resistor_SMD:R_0402_1005Metric" (id 2) (at 58.42 152.4 0)
       (effects (font (size 1.27 1.27)) hide)
@@
   )
   (symbol (lib_id "Transistor_FET:2N7002") (at 65.405 125.73 0) (unit 1)
-    (in_bom yes) (on_board yes) (fields_autoplaced)
-    (property "Reference" "Q5" (id 0) (at 71.755 124.4599 0)
-      (effects (font (size 1.27 1.27)) (justify left))
-    )
-    (property "Value" "2N7002" (id 1) (at 71.755 126.9999 0)
+    (in_bom yes) (on_board yes)
+    (property "Reference" "Q5" (id 0) (at 70.485 124.46 0)
+      (effects (font (size 1.27 1.27)) (justify left))
+    )
+    (property "Value" "AP1606" (id 1) (at 70.485 127 0)
       (effects (font (size 1.27 1.27)) (justify left))
     )
@@
   (symbol (lib_id "Device:R_Small") (at 201.295 132.08 0) (mirror y) (unit 1)
     (in_bom yes) (on_board yes)
-    (property "Reference" "R26" (id 0) (at 198.755 132.715 0))
-    (property "Value" "5.1k" (id 1) (at 198.12 130.81 0))
+    (property "Reference" "R26" (id 0) (at 198.12 130.81 0))
+    (property "Value" "5.1k" (id 1) (at 198.12 133.35 0))
     (property "Footprint" "Resistor_SMD:R_0402_1005Metric" (id 2) (at 201.295 132.08 0)
       (effects (font (size 1.27 1.27)) hide)
@@
   (symbol (lib_id "Device:R_Small") (at 47.625 152.4 0) (unit 1)
     (in_bom yes) (on_board yes)
-    (property "Reference" "R11" (id 0) (at 50.165 153.035 0))
-    (property "Value" "5.1k" (id 1) (at 50.8 151.13 0))
+    (property "Reference" "R11" (id 0) (at 50.8 151.13 0))
+    (property "Value" "5.1k" (id 1) (at 50.8 153.67 0))
     (property "Footprint" "Resistor_SMD:R_0402_1005Metric" (id 2) (at 47.625 152.4 0)
       (effects (font (size 1.27 1.27)) hide)
@@
   (symbol (lib_id "Device:R_Small") (at 39.37 116.205 0) (unit 1)
     (in_bom yes) (on_board yes)
-    (property "Reference" "R8" (id 0) (at 41.91 116.84 0))
-    (property "Value" "220k" (id 1) (at 42.545 114.935 0))
+    (property "Reference" "R8" (id 0) (at 42.545 114.935 0))
+    (property "Value" "220k" (id 1) (at 43.18 117.475 0))
     (property "Footprint" "Resistor_SMD:R_0402_1005Metric" (id 2) (at 39.37 116.205 0)
       (effects (font (size 1.27 1.27)) hide)
@@
   (symbol (lib_id "Device:R_Small") (at 48.26 116.205 0) (unit 1)
     (in_bom yes) (on_board yes)
-    (property "Reference" "R12" (id 0) (at 50.8 116.84 0))
-    (property "Value" "5.1k" (id 1) (at 51.435 114.935 0))
+    (property "Reference" "R12" (id 0) (at 51.435 114.935 0))
+    (property "Value" "5.1k" (id 1) (at 51.435 117.475 0))
     (property "Footprint" "Resistor_SMD:R_0402_1005Metric" (id 2) (at 48.26 116.205 0)
       (effects (font (size 1.27 1.27)) hide)
@@
   )
   (symbol (lib_id "Transistor_FET:2N7002") (at 45.085 161.925 0) (unit 1)
-    (in_bom yes) (on_board yes) (fields_autoplaced)
-    (property "Reference" "Q1" (id 0) (at 51.435 160.6549 0)
-      (effects (font (size 1.27 1.27)) (justify left))
-    )
-    (property "Value" "2N7002" (id 1) (at 51.435 163.1949 0)
+    (in_bom yes) (on_board yes)
+    (property "Reference" "Q1" (id 0) (at 50.165 160.655 0)
+      (effects (font (size 1.27 1.27)) (justify left))
+    )
+    (property "Value" "AP1606" (id 1) (at 50.165 163.195 0)
       (effects (font (size 1.27 1.27)) (justify left))
     )
@@
   (symbol (lib_id "Device:R_Small") (at 67.945 116.205 0) (unit 1)
     (in_bom yes) (on_board yes)
-    (property "Reference" "R25" (id 0) (at 70.485 116.84 0))
-    (property "Value" "5.1k" (id 1) (at 71.12 114.935 0))
+    (property "Reference" "R25" (id 0) (at 71.12 114.935 0))
+    (property "Value" "5.1k" (id 1) (at 71.12 117.475 0))
     (property "Footprint" "Resistor_SMD:R_0402_1005Metric" (id 2) (at 67.945 116.205 0)
       (effects (font (size 1.27 1.27)) hide)
@@
   )
   (symbol (lib_id "Transistor_FET:2N7002") (at 184.15 141.605 0) (mirror y) (unit 1)
-    (in_bom yes) (on_board yes) (fields_autoplaced)
-    (property "Reference" "Q3" (id 0) (at 177.8 140.3349 0)
-      (effects (font (size 1.27 1.27)) (justify left))
-    )
-    (property "Value" "2N7002" (id 1) (at 177.8 142.8749 0)
+    (in_bom yes) (on_board yes)
+    (property "Reference" "Q3" (id 0) (at 178.435 140.335 0)
+      (effects (font (size 1.27 1.27)) (justify left))
+    )
+    (property "Value" "AP1606" (id 1) (at 178.435 142.875 0)
       (effects (font (size 1.27 1.27)) (justify left))
     )
@@
   (symbol (lib_id "Device:R_Small") (at 38.735 152.4 0) (unit 1)
     (in_bom yes) (on_board yes)
-    (property "Reference" "R7" (id 0) (at 41.275 153.035 0))
-    (property "Value" "220k" (id 1) (at 41.91 151.13 0))
+    (property "Reference" "R7" (id 0) (at 41.91 151.13 0))
+    (property "Value" "220k" (id 1) (at 42.545 153.67 0))
     (property "Footprint" "Resistor_SMD:R_0402_1005Metric" (id 2) (at 38.735 152.4 0)
       (effects (font (size 1.27 1.27)) hide)
@@
   (symbol (lib_id "Device:R_Small") (at 59.055 116.205 0) (unit 1)
     (in_bom yes) (on_board yes)
-    (property "Reference" "R21" (id 0) (at 61.595 116.84 0))
-    (property "Value" "220k" (id 1) (at 62.23 114.935 0))
+    (property "Reference" "R21" (id 0) (at 62.23 114.935 0))
+    (property "Value" "220k" (id 1) (at 62.865 117.475 0))
     (property "Footprint" "Resistor_SMD:R_0402_1005Metric" (id 2) (at 59.055 116.205 0)
       (effects (font (size 1.27 1.27)) hide)
@@
   )
   (symbol (lib_id "Transistor_FET:2N7002") (at 64.77 161.925 0) (unit 1)
-    (in_bom yes) (on_board yes) (fields_autoplaced)
-    (property "Reference" "Q4" (id 0) (at 71.12 160.6549 0)
-      (effects (font (size 1.27 1.27)) (justify left))
-    )
-    (property "Value" "2N7002" (id 1) (at 71.12 163.1949 0)
+    (in_bom yes) (on_board yes)
+    (property "Reference" "Q4" (id 0) (at 69.85 160.655 0)
+      (effects (font (size 1.27 1.27)) (justify left))
+    )
+    (property "Value" "AP1606" (id 1) (at 69.85 163.195 0)
       (effects (font (size 1.27 1.27)) (justify left))
     )
@@
   (symbol (lib_id "Device:R_Small") (at 190.5 132.08 0) (mirror y) (unit 1)
     (in_bom yes) (on_board yes)
-    (property "Reference" "R27" (id 0) (at 187.96 132.715 0))
-    (property "Value" "220k" (id 1) (at 187.325 130.81 0))
+    (property "Reference" "R27" (id 0) (at 187.325 130.81 0))
+    (property "Value" "220k" (id 1) (at 186.69 133.35 0))
     (property "Footprint" "Resistor_SMD:R_0402_1005Metric" (id 2) (at 190.5 132.08 0)
       (effects (font (size 1.27 1.27)) hide)
@@
   (symbol (lib_id "Device:R_Small") (at 210.185 132.08 0) (mirror y) (unit 1)
     (in_bom yes) (on_board yes)
-    (property "Reference" "R28" (id 0) (at 207.645 132.715 0))
-    (property "Value" "220k" (id 1) (at 207.01 130.81 0))
+    (property "Reference" "R28" (id 0) (at 207.01 130.81 0))
+    (property "Value" "220k" (id 1) (at 206.375 133.35 0))
     (property "Footprint" "Resistor_SMD:R_0402_1005Metric" (id 2) (at 210.185 132.08 0)
       (effects (font (size 1.27 1.27)) hide)
@@
   )
   (symbol (lib_id "Transistor_FET:2N7002") (at 203.835 141.605 0) (mirror y) (unit 1)
-    (in_bom yes) (on_board yes) (fields_autoplaced)
-    (property "Reference" "Q6" (id 0) (at 197.485 140.3349 0)
-      (effects (font (size 1.27 1.27)) (justify left))
-    )
-    (property "Value" "2N7002" (id 1) (at 197.485 142.8749 0)
+    (in_bom yes) (on_board yes)
+    (property "Reference" "Q6" (id 0) (at 198.755 140.335 0)
+      (effects (font (size 1.27 1.27)) (justify left))
+    )
+    (property "Value" "AP1606" (id 1) (at 198.755 142.875 0)
       (effects (font (size 1.27 1.27)) (justify left))
     )
@@
   )
   (symbol (lib_id "Transistor_FET:2N7002") (at 45.72 125.73 0) (unit 1)
-    (in_bom yes) (on_board yes) (fields_autoplaced)
-    (property "Reference" "Q2" (id 0) (at 52.07 124.4599 0)
-      (effects (font (size 1.27 1.27)) (justify left))
-    )
-    (property "Value" "2N7002" (id 1) (at 52.07 126.9999 0)
-      (effects (font (size 1.27 1.27)) (justify left))
-    )
+    (in_bom yes) (on_board yes)
+    (property "Reference" "Q2" (id 0) (at 50.8 124.46 0)
+      (effects (font (size 1.27 1.27)) (justify left))
+    )
+    (property "Value" "AP1606" (id 1) (at 50.8 127 0)
+      (effects (font (size 1.27 1.27)) (justify left))
+    )

Commit message: update footprints + render + power pull-ups
Parts:
- R20, R21, R27, R28, R7, R8: value 220k -> 47k
