File: KiCad/h_usb3_switching.kicad_sch (KiCad schematic)
At the start: 3 parts, among them U1 FUSB340TMX, U2 FUSB340TMX

Commit message: Use 0603 resistors and capacitors
Parts:
- R6: footprint Resistor_SMD:R_0805_2012Metric -> Resistor_SMD:R_0603_1608Metric
Changed lines of the file:
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@@
       (effects (font (size 1.27 1.27)) (justify left))
     )
-    (property "Footprint" "Resistor_SMD:R_0805_2012Metric" (id 2) (at 64.77 91.44 0)
+    (property "Footprint" "Resistor_SMD:R_0603_1608Metric" (id 2) (at 64.77 91.44 0)
       (effects (font (size 1.27 1.27)) hide)
     )
